Commit message: feature: added camera and world

File: urdf/materials.xacro (robot description, xacro)
@@ -31,3 +31,8 @@
         </material>
     </xacro:macro>
+    <xacro:macro name="green_material">
+        <material name="green">
+            <color rgba="0.0 1.0 0.0 1.0"/>
+        </material>
+    </xacro:macro>
 </robot>

File: urdf/waver.xacro (robot description, xacro)
@@ -7,4 +7,5 @@
   <xacro:include filename="$(find waver_description)/urdf/lidar.xacro" />
   <xacro:include filename="$(find waver_description)/urdf/imu.xacro" />
+  <xacro:include filename="$(find waver_description)/urdf/camera.xacro" />
   <!-- ******************************* Links ******************************* -->
   <link name="base_footprint"></link>
