Commit message: feature: support for gazebo

File: urdf/imu.xacro (robot description, xacro)
@@ -12,5 +12,5 @@
             <origin xyz="${position_imu}" rpy="0 0 ${pi/2}" />
             <geometry>
-                <mesh filename="package://waver_description/meshes/board_link.stl" scale="${scale}" />
+                <mesh filename="file:///$(find waver_description)/meshes/board_link.stl" scale="${scale}" />
             </geometry>
             <xacro:dark_green_material />
@@ -19,5 +19,5 @@
             <origin xyz="${position_imu}" rpy="0 0 ${pi/2}" />
             <geometry>
-                <mesh filename="package://waver_description/meshes/board_link.stl" scale="${scale}" />
+                <mesh filename="file:///$(find waver_description)/meshes/board_link.stl" scale="${scale}" />
             </geometry>
         </collision>
@@ -28,24 +28,24 @@
         <child link="imu_link" />
     </joint>
-    <gazebo reference="imu_link">
-        <material>Gazebo/Orange</material>
-        <gravity>true</gravity>
+    <!-- <gazebo reference="imu_link">
         <sensor name="imu_sensor" type="imu">
             <always_on>true</always_on>
             <update_rate>100</update_rate>
             <visualize>true</visualize>
-            <topic>imu</topic>
-            <plugin filename="libgazebo_ros_imu_sensor.so" name="imu_plugin">
-                <topicName>imu</topicName>
-                <bodyName>imu_link</bodyName>
-                <updateRateHZ>10.0</updateRateHZ>
-                <gaussianNoise>0.0</gaussianNoise>
-                <xyzOffset>0 0 0</xyzOffset>
-                <rpyOffset>0 0 0</rpyOffset>
-                <frameName>imu_link</frameName>
-                <initialOrientationAsReference>false</initialOrientationAsReference>
+            <plugin filename="libgazebo_ros_imu_sensor.so" name="gazebo_ros_imu_sensor">
+                <ros>
+                    <namespace></namespace>
+                    <remapping>imu:=imu/data_raw</remapping>
+                </ros>
+                <frame_name>imu_link</frame_name>
+                <update_rate>100.0</update_rate>
+                <orientation_reference_frame>world</orientation_reference_frame>
+                <imu_parameters>
+                    <noise_density>0.0025</noise_density>
+                    <bias_correlation_time>1000000.0</bias_correlation_time>
+                    <random_walk>0.0002</random_walk>
+                </imu_parameters>
             </plugin>
-            <pose>0 0 0 0 0 0</pose>
         </sensor>
-    </gazebo>
+    </gazebo> -->
 </robot>

File: urdf/lidar.xacro (robot description, xacro)
@@ -13,5 +13,5 @@
             <origin xyz="0 0 -0.027" rpy="0 0 ${pi/2}" />
             <geometry>
-                <mesh filename="package://waver_description/meshes/LD19.stl" scale="${scale}" />
+                <mesh filename="file:///$(find waver_description)/meshes/LD19.stl" scale="${scale}" />
             </geometry>
             <xacro:black_material />
@@ -20,5 +20,5 @@
             <origin xyz="0 0 -0.027" rpy="0 0 ${pi/2}" />
             <geometry>
-                <mesh filename="package://waver_description/meshes/LD19.stl" scale="${scale}" />
+                <mesh filename="file:///$(find waver_description)/meshes/LD19.stl" scale="${scale}" />
             </geometry>
         </collision>
@@ -41,4 +41,5 @@
                     <horizontal>
                         <samples>${lidar_samples}</samples>
+                        <resolution>1</resolution>
                         <min_angle>${lidar_min_angle}</min_angle>
                         <max_angle>${lidar_max_angle}</max_angle>
@@ -49,13 +50,12 @@
                     <max>${lidar_max_range}</max>
                 </range>
-                <noise>
-                    <type>gaussian</type>
-                    <mean>0.0</mean>
-                    <stddev>0.01</stddev>
-                </noise>
             </ray>
-            <plugin name="lidar_controller" filename="libgazebo_ros_laser.so">
-                <topicName>scan</topicName>
-                <frameName>lidar_link</frameName>
+            <plugin name="gazebo_ros_laser_controller" filename="libgazebo_ros_ray_sensor.so">
+                <ros>
+                    <namespace/>
+                    <argument>--ros-args --remap __ns:=/</argument>
+                    <argument>--ros-args --remap scan:=scan</argument>
+                </ros>
+                <frameName>${lidar_link}</frameName>
             </plugin>
         </sensor>

File: urdf/waver.gazebo.xacro (robot description, xacro)
@@ -62,27 +62,27 @@
     <material>Gazebo/Black</material>
   </gazebo>
-  <gazebo>
-    <plugin name="skid_steer_drive_controller" filename="libgazebo_ros_skid_steer_drive.so">
-      <robotNamespace></robotNamespace>
-      <updateRate>100.0</updateRate>
-      <leftFrontJoint>wheel_front_left_joint</leftFrontJoint>
-      <rightFrontJoint>wheel_front_right_joint</rightFrontJoint>
-      <leftRearJoint>wheel_back_left_joint</leftRearJoint>
-      <rightRearJoint>wheel_back_right_joint</rightRearJoint>
-      <wheelSeparation>${wheel_separation}</wheelSeparation>
-      <wheelDiameter>${2*wheel_radius}</wheelDiameter>
-      <torque>2</torque>
-      <commandTopic>cmd_vel</commandTopic>
-      <odometryTopic>odom</odometryTopic>
-      <odometryFrame>odom</odometryFrame>
-      <robotBaseFrame>base_footprint</robotBaseFrame>
-      <publishWheelTF>true</publishWheelTF>
-      <publishOdom>true</publishOdom>
-      <publishWheelJointState>true</publishWheelJointState>
-      <covariance_x>0.0001</covariance_x>
-      <covariance_y>0.0001</covariance_y>
-      <covariance_yaw>0.01</covariance_yaw>
-      <broadcastTF>true</broadcastTF>
-    </plugin>
-  </gazebo>
+    <!-- <gazebo>
+      <plugin name="diff_drive_controller" filename="libgazebo_ros_diff_drive.so">
+        <ros>
+          <namespace></namespace>
+          <remapping>cmd_vel:=cmd_vel</remapping>
+        </ros>
+        <update_rate>100.0</update_rate>
+        <left_joint>wheel_front_left_joint</left_joint>
+        <right_joint>wheel_front_right_joint</right_joint>
+        <wheel_separation>${wheel_separation}</wheel_separation>
+        <wheel_diameter>${wheel_radius * 2}</wheel_diameter>
+        <robot_base_frame>base_footprint</robot_base_frame>
+        <odom_frame>odom</odom_frame>
+        <publish_odom>true</publish_odom>
+        <publish_odom_tf>true</publish_odom_tf>
+      </plugin>
+    </gazebo> -->
+    <gazebo>
+      <plugin name="four_wheel_drive_controller" filename="libwaver_description.so">
+        <ros>
+          <argument>cmd_vel:=/cmd_vel</argument>
+        </ros>
+      </plugin>
+    </gazebo>
 </robot>

File: urdf/waver.xacro (robot description, xacro)
@@ -3,8 +3,8 @@
   <xacro:include filename="$(find waver_description)/urdf/materials.xacro" />
   <xacro:include filename="$(find waver_description)/urdf/util.xacro" />
-  <xacro:include filename="$(find waver_description)/urdf/waver.trans.xacro" />
+  <!-- <xacro:include filename="$(find waver_description)/urdf/waver.trans.xacro" /> -->
   <xacro:include filename="$(find waver_description)/urdf/waver.gazebo.xacro" />
-  <xacro:include filename="$(find waver_description)/urdf/lidar.xacro" />
-  <xacro:include filename="$(find waver_description)/urdf/imu.xacro" />
+  <!-- <xacro:include filename="$(find waver_description)/urdf/lidar.xacro" /> -->
+  <!-- <xacro:include filename="$(find waver_description)/urdf/imu.xacro" /> -->
   <!-- ******************************* Links ******************************* -->
   <link name="base_footprint"></link>
@@ -18,5 +18,5 @@
       <origin xyz="0 0 0" rpy="0 0 ${pi/2}" />
       <geometry>
-        <mesh filename="package://waver_description/meshes/base_link.stl" scale="${scale}" />
+        <mesh filename="file:///$(find waver_description)/meshes/base_link.stl" scale="${scale}" />
       </geometry>
       <xacro:dark_gray_material />
@@ -25,5 +25,5 @@
       <origin xyz="0 0 0" rpy="0 0 ${pi/2}" />
       <geometry>
-        <mesh filename="package://waver_description/meshes/base_link.stl" scale="${scale}" />
+        <mesh filename="file:///$(find waver_description)/meshes/base_link.stl" scale="${scale}" />
       </geometry>
     </collision>
@@ -38,5 +38,5 @@
       <origin xyz="0 0 0" rpy="0 0 ${pi/2}" />
       <geometry>
-        <mesh filename="package://waver_description/meshes/top_shell_link.stl" scale="${scale}" />
+        <mesh filename="file:///$(find waver_description)/meshes/top_shell_link.stl" scale="${scale}" />
       </geometry>
       <xacro:dark_gray_material />
@@ -45,5 +45,5 @@
       <origin xyz="0 0 0" rpy="0 0 ${pi/2}" />
       <geometry>
-        <mesh filename="package://waver_description/meshes/top_shell_link.stl" scale="${scale}" />
+        <mesh filename="file:///$(find waver_description)/meshes/top_shell_link.stl" scale="${scale}" />
       </geometry>
     </collision>
@@ -58,5 +58,5 @@
       <origin xyz="${position_acces}" rpy="0 0 ${pi/2}" />
       <geometry>
-        <mesh filename="package://waver_description/meshes/accessories_link.stl" scale="${scale}" />
+        <mesh filename="file:///$(find waver_description)/meshes/accessories_link.stl" scale="${scale}" />
       </geometry>
       <xacro:black_material />
@@ -65,5 +65,5 @@
       <origin xyz="${position_acces}" rpy="0 0 ${pi/2}" />
       <geometry>
-        <mesh filename="package://waver_description/meshes/accessories_link.stl" scale="${scale}" />
+        <mesh filename="file:///$(find waver_description)/meshes/accessories_link.stl" scale="${scale}" />
       </geometry>
     </collision>
@@ -78,5 +78,5 @@
       <origin xyz="${position_acces1}" rpy="0 0 ${pi/2}" />
       <geometry>
-        <mesh filename="package://waver_description/meshes/accessories1_link.stl" scale="${scale}" />
+        <mesh filename="file:///$(find waver_description)/meshes/accessories1_link.stl" scale="${scale}" />
       </geometry>
       <xacro:black_material />
@@ -85,5 +85,5 @@
       <origin xyz="${position_acces1}" rpy="0 0 ${pi/2}" />
       <geometry>
-        <mesh filename="package://waver_description/meshes/accessories1_link.stl" scale="${scale}" />
+        <mesh filename="file:///$(find waver_description)/meshes/accessories1_link.stl" scale="${scale}" />
       </geometry>
     </collision>
@@ -98,5 +98,5 @@
       <origin xyz="${position_screen}" rpy="0 0 ${pi/2}" />
       <geometry>
-        <mesh filename="package://waver_description/meshes/oled_screen_link.stl" scale="${scale}" />
+        <mesh filename="file:///$(find waver_description)/meshes/oled_screen_link.stl" scale="${scale}" />
       </geometry>
       <xacro:dark_blue_material />
@@ -105,5 +105,5 @@
       <origin xyz="${position_screen}" rpy="0 0 ${pi/2}" />
       <geometry>
-        <mesh filename="package://waver_description/meshes/oled_screen_link.stl" scale="${scale}" />
+        <mesh filename="file:///$(find waver_description)/meshes/oled_screen_link.stl" scale="${scale}" />
       </geometry>
     </collision>
@@ -118,5 +118,5 @@
       <origin xyz="${position_wbl}" rpy="0 0 ${pi/2}" />
       <geometry>
-        <mesh filename="package://waver_description/meshes/wheel_back_left_link.stl" scale="${scale}" />
+        <mesh filename="file:///$(find waver_description)/meshes/wheel_back_left_link.stl" scale="${scale}" />
       </geometry>
       <xacro:black_material />
@@ -125,5 +125,5 @@
       <origin xyz="${position_wbl}" rpy="0 0 ${pi/2}" />
       <geometry>
-        <mesh filename="package://waver_description/meshes/wheel_back_left_link.stl" scale="${scale}" />
+        <mesh filename="file:///$(find waver_description)/meshes/wheel_back_left_link.stl" scale="${scale}" />
       </geometry>
     </collision>
@@ -138,5 +138,5 @@
       <origin xyz="${position_wfl}" rpy="0 0 ${pi/2}" />
       <geometry>
-        <mesh filename="package://waver_description/meshes/wheel_front_left_link.stl" scale="${scale}" />
+        <mesh filename="file:///$(find waver_description)/meshes/wheel_front_left_link.stl" scale="${scale}" />
       </geometry>
       <xacro:black_material />
@@ -145,5 +145,5 @@
       <origin xyz="${position_wfl}" rpy="0 0 ${pi/2}" />
       <geometry>
-        <mesh filename="package://waver_description/meshes/wheel_front_left_link.stl" scale="${scale}" />
+        <mesh filename="file:///$(find waver_description)/meshes/wheel_front_left_link.stl" scale="${scale}" />
       </geometry>
     </collision>
@@ -158,5 +158,5 @@
       <origin xyz="${position_wfr}" rpy="0 0 ${pi/2}" />
       <geometry>
-        <mesh filename="package://waver_description/meshes/wheel_front_right_link.stl" scale="${scale}" />
+        <mesh filename="file:///$(find waver_description)/meshes/wheel_front_right_link.stl" scale="${scale}" />
       </geometry>
       <xacro:black_material />
@@ -165,5 +165,5 @@
       <origin xyz="${position_wfr}" rpy="0 0 ${pi/2}" />
       <geometry>
-        <mesh filename="package://waver_description/meshes/wheel_front_right_link.stl" scale="${scale}" />
+        <mesh filename="file:///$(find waver_description)/meshes/wheel_front_right_link.stl" scale="${scale}" />
       </geometry>
     </collision>
@@ -178,5 +178,5 @@
       <origin xyz="${position_wbr}" rpy="0 0 ${pi/2}" />
       <geometry>
-        <mesh filename="package://waver_description/meshes/wheel_back_right_link.stl" scale="${scale}" />
+        <mesh filename="file:///$(find waver_description)/meshes/wheel_back_right_link.stl" scale="${scale}" />
       </geometry>
       <xacro:black_material />
@@ -185,5 +185,5 @@
       <origin xyz="${position_wbr}" rpy="0 0 ${pi/2}" />
       <geometry>
-        <mesh filename="package://waver_description/meshes/wheel_back_right_link.stl" scale="${scale}" />
+        <mesh filename="file:///$(find waver_description)/meshes/wheel_back_right_link.stl" scale="${scale}" />
       </geometry>
     </collision>

Commit message: chore: updated xacro files

File: urdf/imu.xacro (robot description, xacro)
@@ -29,5 +29,5 @@
     </joint>
     <gazebo reference="imu_link">
-        <sensor name="imu_sensor" type="imu">
+        <!-- <sensor name="imu_sensor" type="imu">
             <always_on>true</always_on>
             <update_rate>100</update_rate>
@@ -47,4 +47,16 @@
                 </imu_parameters>
             </plugin>
+        </sensor> -->
+        <sensor name="imu_sensor" type="imu">
+        <!-- ensure the sensor is active (required) -->
+        <always_on>true</always_on>
+        <update_rate>50</update_rate>
+        <plugin name="my_imu_plugin" filename="libgazebo_ros_imu_sensor.so">
+            <ros>
+            <!-- publish to /imu/data -->
+            <namespace>/imu</namespace>
+            <remapping>~/out:=data</remapping>
+            </ros>
+        </plugin>
         </sensor>
     </gazebo>

File: urdf/util.xacro (robot description, xacro)
@@ -12,5 +12,5 @@
     <xacro:property name="pos_y_base" value="-6.582658272236586e-06" />
     <xacro:property name="pos_z_base" value="0.002703800678253174" />
-    <xacro:property name="mass_base" value="0.37038398045076265" />
+    <xacro:property name="mass_base" value="1.37038398045076265" />
     <xacro:property name="mass_center_base" value="${pos_x_base} ${pos_y_base} ${pos_z_base}" />
     <xacro:property name="position_base" value="${-pos_x_base} ${-pos_y_base} ${-pos_z_base}" />
@@ -77,5 +77,5 @@
     <xacro:property name="pos_y_wfr" value="-0.048593093872070316" />
     <xacro:property name="pos_z_wfr" value="0.004798998355865478" />
-    <xacro:property name="mass_wfr" value="1.0170112199417978" />
+    <xacro:property name="mass_wfr" value="1.0170123141691128" />
     <xacro:property name="mass_center_wfr" value="${pos_x_wfr} ${pos_y_wfr} ${pos_z_wfr}" />
     <xacro:property name="position_wfr" value="${pos_y_wfr} ${-pos_x_wfr} ${-pos_z_wfr}" />

File: urdf/waver.gazebo.xacro (robot description, xacro)
@@ -86,5 +86,5 @@
         <!-- <publish_wheel_tf>true</publish_wheel_tf> -->
         <!-- <publish_wheel_joint_state>true</publish_wheel_joint_state> -->
-        <torque>15.0</torque>
+        <torque>30.0</torque>
       </plugin>
     </gazebo>

File: urdf/waver.xacro (robot description, xacro)
@@ -6,5 +6,5 @@
   <xacro:include filename="$(find waver_description)/urdf/waver.gazebo.xacro" />
   <xacro:include filename="$(find waver_description)/urdf/lidar.xacro" />
-  <!-- <xacro:include filename="$(find waver_description)/urdf/imu.xacro" /> -->
+  <xacro:include filename="$(find waver_description)/urdf/imu.xacro" />
   <!-- ******************************* Links ******************************* -->
   <link name="base_footprint"></link>
@@ -113,5 +113,5 @@
       <mass value="${mass_wbl}" />
       <origin xyz="0 0 0" rpy="0 0 ${pi/2}" />
-      <inertia ixx="0.0011153598236428852" iyy="0.0007115715200341761" izz="0.0007099489264864056" ixy="0.0" iyz="0.0" ixz="0.0" />
+      <inertia ixx="0.0011153598236428852" iyy="0.0007115715475157099" izz="0.0007099489539679392" ixy="0.0" iyz="0.0" ixz="0.0" />
     </inertial>
     <visual>
@@ -133,5 +133,5 @@
       <mass value="${mass_wfl}" />
       <origin xyz="0 0 0" rpy="0 0 ${pi/2}" />
-      <inertia ixx="0.0011153873944048257" iyy="0.0007115715200341761" izz="0.0007099764972483459" ixy="0.0" iyz="0.0" ixz="0.0" />
+      <inertia ixx="0.0011153598236428852" iyy="0.0007115715475157099" izz="0.0007099489539679392" ixy="0.0" iyz="0.0" ixz="0.0" />
     </inertial>
     <visual>
@@ -173,5 +173,5 @@
       <mass value="${mass_wbr}" />
       <origin xyz="0 0 0" rpy="0 0 ${pi/2}" />
-      <inertia ixx="0.0011153873944048257" iyy="0.0007115715475157099" izz="0.0007099765247298796" ixy="0.0" iyz="0.0" ixz="0.0" />
+      <inertia ixx="0.0011153598236428852" iyy="0.0007115715475157099" izz="0.0007099489539679392" ixy="0.0" iyz="0.0" ixz="0.0" />
     </inertial>
     <visual>
@@ -229,14 +229,14 @@
   </joint>
   <joint name="wheel_front_right_joint" type="continuous">
-    <origin xyz="${position_wfr_joint}" rpy="0 0 ${pi}" />
+    <origin xyz="${position_wfr_joint}" rpy="0 0 0" />
     <parent link="base_link" />
     <child link="wheel_front_right_link" />
-    <axis xyz="0 -1 0" />
+    <axis xyz="0 1 0" />
   </joint>
   <joint name="wheel_back_right_joint" type="continuous">
-    <origin xyz="${position_wbr_joint}" rpy="0 0 ${pi}" />
+    <origin xyz="${position_wbr_joint}" rpy="0 0 0" />
     <parent link="base_link" />
     <child link="wheel_back_right_link" />
-    <axis xyz="0 -1 0" />
+    <axis xyz="0 1 0" />
   </joint>
 </robot>
