Commit message: chore: mass and inertia updated

File: urdf/imu.xacro (robot description, xacro)
@@ -7,5 +7,5 @@
             <mass value="${mass_imu}" />
             <origin xyz="${mass_center_imu}" rpy="0 0 ${pi/2}" />
-            <inertia ixx="5.313564367625195e-06" iyy="5.192849578266062e-06" izz="8.832425081682543e-06" ixy="0.0" iyz="0.0" ixz="0.0" />
+            <inertia ixx="4.297064285474092e-13" iyy="4.199442581059605e-13" izz="7.142756866533696e-13" ixy="0.0" iyz="0.0" ixz="0.0" />
         </inertial>
         <visual>

File: urdf/lidar.xacro (robot description, xacro)
@@ -7,6 +7,5 @@
             <mass value="${mass_lidar}" />
             <origin xyz="0 0 0" rpy="0 0 0" />
-            <inertia ixx="1.3010226e-05" iyy="1.6209553e-05" izz="2.1055697e-05" ixy="0.0" iyz="0.0"
-                ixz="0.0" />
+            <inertia ixx="1.1969407982864896e-05" iyy="1.4912788506851203e-05" izz="1.9371239273809308e-05" ixy="0.0" iyz="0.0" ixz="0.0" />
         </inertial>
         <visual>

File: urdf/util.xacro (robot description, xacro)
@@ -12,5 +12,5 @@
     <xacro:property name="pos_y_base" value="-6.582658272236586e-06" />
     <xacro:property name="pos_z_base" value="0.002703800678253174" />
-    <xacro:property name="mass_base" value="1.37038398045076265" />
+    <xacro:property name="mass_base" value="0.110" />
     <xacro:property name="mass_center_base" value="${pos_x_base} ${pos_y_base} ${pos_z_base}" />
     <xacro:property name="position_base" value="${-pos_x_base} ${-pos_y_base} ${-pos_z_base}" />
@@ -19,5 +19,5 @@
     <xacro:property name="pos_y_top" value="-0.0006833337545394898" />
     <xacro:property name="pos_z_top" value="0.038709537506103515" />
-    <xacro:property name="mass_top" value="0.7277708834628859" />
+    <xacro:property name="mass_top" value="0.326" />
     <xacro:property name="mass_center_top" value="${pos_x_top} ${pos_y_top} ${pos_z_top}" />
     <xacro:property name="position_top" value="${-pos_x_top} ${-pos_y_top} ${-pos_z_top}" />
@@ -26,32 +26,32 @@
     <xacro:property name="pos_y_acces" value="0.08693458557128907" />
     <xacro:property name="pos_z_acces" value="0.04861989974975586" />
-    <xacro:property name="mass_acces" value="0.0017616158924187116" />
+    <xacro:property name="mass_acces" value="0.000000001" />
     <xacro:property name="mass_center_acces" value="${pos_x_acces} ${pos_y_acces} ${pos_z_acces}" />
     <xacro:property name="position_acces" value="${pos_y_acces} ${-pos_x_acces} ${-pos_z_acces}" />
-    <xacro:property name="positions_acces_joint" value="${-pos_y_acces} ${pos_x_acces} ${pos_z_acces}"/>
+    <xacro:property name="positions_acces_joint" value="${-pos_y_acces} ${pos_x_acces} ${pos_z_acces}" />
     <!-- Accessories1 specifications -->
     <xacro:property name="pos_x_acces1" value="-0.002510018587112427" />
     <xacro:property name="pos_y_acces1" value="0.07360986328125002" />
     <xacro:property name="pos_z_acces1" value="0.035275302886962887" />
-    <xacro:property name="mass_acces1" value="0.0021489822783274555" />
+    <xacro:property name="mass_acces1" value="0.000000001" />
     <xacro:property name="mass_center_acces1" value="${pos_x_acces1} ${pos_y_acces1} ${pos_z_acces1}" />
     <xacro:property name="position_acces1" value="${pos_y_acces1} ${-pos_x_acces1} ${-pos_z_acces1}" />
-    <xacro:property name="positions_acces1_joint" value="${-pos_y_acces1} ${pos_x_acces1} ${pos_z_acces1}"/>
+    <xacro:property name="positions_acces1_joint" value="${-pos_y_acces1} ${pos_x_acces1} ${pos_z_acces1}" />
     <!-- IMU speficications -->
     <xacro:property name="pos_x_imu" value="-0.009815516471862793" />
     <xacro:property name="pos_y_imu" value="0.009279213905334474" />
     <xacro:property name="pos_z_imu" value="0.04129100418090821" />
-    <xacro:property name="mass_imu" value="0.012365568710683028" />
+    <xacro:property name="mass_imu" value="0.000000001" />
     <xacro:property name="mass_center_imu" value="${pos_x_imu} ${pos_y_imu} ${pos_z_imu}" />
     <xacro:property name="position_imu" value="${pos_y_imu} ${-pos_x_imu} ${-pos_z_imu}" />
-    <xacro:property name="positions_imu_joint" value="${-pos_y_imu} ${pos_x_imu} ${pos_z_imu}"/>
+    <xacro:property name="positions_imu_joint" value="${-pos_y_imu} ${pos_x_imu} ${pos_z_imu}" />
     <!-- Oled Screen speficications -->
     <xacro:property name="pos_x_screen" value="-6.735318456776441e-07" />
     <xacro:property name="pos_y_screen" value="0.05096461868286133" />
     <xacro:property name="pos_z_screen" value="0.048232952117919926" />
-    <xacro:property name="mass_screen" value="0.0014091265350616076" />
+    <xacro:property name="mass_screen" value="0.000000001" />
     <xacro:property name="mass_center_screen" value="${pos_x_screen} ${pos_y_screen} ${pos_z_screen}" />
     <xacro:property name="position_screen" value="${pos_y_screen} ${-pos_x_screen} ${-pos_z_screen}" />
-    <xacro:property name="positions_screen_joint" value="${-pos_y_screen} ${pos_x_screen} ${pos_z_screen}"/>
+    <xacro:property name="positions_screen_joint" value="${-pos_y_screen} ${pos_x_screen} ${pos_z_screen}" />
     <!-- Wheels specifications -->
     <xacro:property name="wheel_separation" value="123e-3" />
@@ -61,34 +61,34 @@
     <xacro:property name="pos_y_wbl" value="0.04859128189086914" />
     <xacro:property name="pos_z_wbl" value="0.004798986434936523" />
-    <xacro:property name="mass_wbl" value="1.01701435808657" />
+    <xacro:property name="mass_wbl" value="0.061" />
     <xacro:property name="mass_center_wbl" value="${pos_x_wbl} ${pos_y_wbl} ${pos_z_wbl}" />
     <xacro:property name="position_wbl" value="${pos_y_wbl} ${-pos_x_wbl} ${-pos_z_wbl}" />
-    <xacro:property name="position_wbl_joint" value="${-pos_y_wbl} ${pos_x_wbl} ${pos_z_wbl}"/>
+    <xacro:property name="position_wbl_joint" value="${-pos_y_wbl} ${pos_x_wbl} ${pos_z_wbl}" />
     <!-- WFL specifications -->
     <xacro:property name="pos_x_wfl" value="0.06538582611083985" />
     <xacro:property name="pos_y_wfl" value="-0.048406845092773446" />
     <xacro:property name="pos_z_wfl" value="0.004799012184143066" />
-    <xacro:property name="mass_wfl" value="1.0170155374515382" />
+    <xacro:property name="mass_wfl" value="0.061" />
     <xacro:property name="mass_center_wfl" value="${pos_x_wfl} ${pos_y_wfl} ${pos_z_wfl}" />
     <xacro:property name="position_wfl" value="${pos_y_wfl} ${-pos_x_wfl} ${-pos_z_wfl}" />
-    <xacro:property name="position_wfl_joint" value="${-pos_y_wfl} ${pos_x_wfl} ${pos_z_wfl}"/>
+    <xacro:property name="position_wfl_joint" value="${-pos_y_wfl} ${pos_x_wfl} ${pos_z_wfl}" />
     <!-- WFR specifications -->
     <xacro:property name="pos_x_wfr" value="-0.06528724670410156" />
     <xacro:property name="pos_y_wfr" value="-0.048593093872070316" />
     <xacro:property name="pos_z_wfr" value="0.004798998355865478" />
-    <xacro:property name="mass_wfr" value="1.0170123141691128" />
+    <xacro:property name="mass_wfr" value="0.061" />
     <xacro:property name="mass_center_wfr" value="${pos_x_wfr} ${pos_y_wfr} ${pos_z_wfr}" />
     <xacro:property name="position_wfr" value="${pos_y_wfr} ${-pos_x_wfr} ${-pos_z_wfr}" />
-    <xacro:property name="position_wfr_joint" value="${-pos_y_wfr} ${pos_x_wfr} ${pos_z_wfr}"/>
+    <xacro:property name="position_wfr_joint" value="${-pos_y_wfr} ${pos_x_wfr} ${pos_z_wfr}" />
     <!-- WBR specifications -->
     <xacro:property name="pos_x_wbr" value="-0.0652872543334961" />
     <xacro:property name="pos_y_wbr" value="0.04840502166748047" />
     <xacro:property name="pos_z_wbr" value="0.004799028396606446" />
-    <xacro:property name="mass_wbr" value="1.0170123141691128" />
+    <xacro:property name="mass_wbr" value="0.061" />
     <xacro:property name="mass_center_wbr" value="${pos_x_wbr} ${pos_y_wbr} ${pos_z_wbr}" />
     <xacro:property name="position_wbr" value="${pos_y_wbr} ${-pos_x_wbr} ${-pos_z_wbr}" />
-    <xacro:property name="position_wbr_joint" value="${-pos_y_wbr} ${pos_x_wbr} ${pos_z_wbr}"/>
+    <xacro:property name="position_wbr_joint" value="${-pos_y_wbr} ${pos_x_wbr} ${pos_z_wbr}" />
     <!-- Lidar specifications -->
-    <xacro:property name="mass_lidar" value="0.05" />
+    <xacro:property name="mass_lidar" value="0.046" />
     <xacro:property name="lidar_model" value="HLS-LFCD-LDS" />
     <xacro:property name="lidar_link" value="lidar_link" />

File: urdf/waver.xacro (robot description, xacro)
@@ -14,10 +14,11 @@
       <mass value="${mass_base}" />
       <origin xyz="${mass_center_base}" rpy="0 0 ${pi/2}" />
-      <inertia ixx="0.0008255973835920386" iyy="0.0005293282898445326" izz="0.0013315199498696443" ixy="0.0" iyz="0.0" ixz="0.0" />
-    </inertial>
-    <visual>
-      <origin xyz="0 0 0" rpy="0 0 ${pi/2}" />
-      <geometry>
-        <mesh filename="file:///$(find waver_description)/meshes/base_link.stl" scale="${scale}" />
+      <inertia ixx="0.00024519341275127564" iyy="0.0001572047252476648" izz="0.0001572047252476648"
+        ixy="0.0" iyz="0.0" ixz="0.0" />
+    </inertial>
+    <visual>
+      <origin xyz="0 0 0" rpy="0 0 ${pi/2}" />
+      <geometry>
+        <mesh filename="package://waver_description/meshes/base_link.stl" scale="${scale}" />
       </geometry>
       <xacro:dark_gray_material />
@@ -26,5 +27,5 @@
       <origin xyz="0 0 0" rpy="0 0 ${pi/2}" />
       <geometry>
-        <mesh filename="file:///$(find waver_description)/meshes/base_link.stl" scale="${scale}" />
+        <mesh filename="package://waver_description/meshes/base_link.stl" scale="${scale}" />
       </geometry>
     </collision>
@@ -34,10 +35,11 @@
       <mass value="${mass_top}" />
       <origin xyz="${mass_center_top}" rpy="0 0 ${pi/2}" />
-      <inertia ixx="0.0022122780308922725" iyy="0.0018048674350663336" izz="0.003659349844340526" ixy="0.0" iyz="0.0" ixz="0.0" />
-    </inertial>
-    <visual>
-      <origin xyz="0 0 0" rpy="0 0 ${pi/2}" />
-      <geometry>
-        <mesh filename="file:///$(find waver_description)/meshes/top_shell_link.stl" scale="${scale}" />
+      <inertia ixx="0.0009909748444994777" iyy="0.0008084780487946392" izz="0.0016391807866491105"
+        ixy="0.0" iyz="0.0" ixz="0.0" />
+    </inertial>
+    <visual>
+      <origin xyz="0 0 0" rpy="0 0 ${pi/2}" />
+      <geometry>
+        <mesh filename="package://waver_description/meshes/top_shell_link.stl" scale="${scale}" />
       </geometry>
       <xacro:dark_gray_material />
@@ -46,5 +48,5 @@
       <origin xyz="0 0 0" rpy="0 0 ${pi/2}" />
       <geometry>
-        <mesh filename="file:///$(find waver_description)/meshes/top_shell_link.stl" scale="${scale}" />
+        <mesh filename="package://waver_description/meshes/top_shell_link.stl" scale="${scale}" />
       </geometry>
     </collision>
@@ -54,10 +56,11 @@
       <mass value="${mass_acces}" />
       <origin xyz="${mass_center_acces}" rpy="0 0 ${pi/2}" />
-      <inertia ixx="2.2622278969724113e-07" iyy="7.36227380617578e-07" izz="7.362274117066844e-07" ixy="0.0" iyz="0.0" ixz="0.0" />
+      <inertia ixx="1.284177729497181e-13" iyy="4.1792730400878273e-13" izz="4.1792732165684473e-13"
+        ixy="0.0" iyz="0.0" ixz="0.0" />
     </inertial>
     <visual>
       <origin xyz="${position_acces}" rpy="0 0 ${pi/2}" />
       <geometry>
-        <mesh filename="file:///$(find waver_description)/meshes/accessories_link.stl" scale="${scale}" />
+        <mesh filename="package://waver_description/meshes/accessories_link.stl" scale="${scale}" />
       </geometry>
       <xacro:black_material />
@@ -66,5 +69,5 @@
       <origin xyz="${position_acces}" rpy="0 0 ${pi/2}" />
       <geometry>
-        <mesh filename="file:///$(find waver_description)/meshes/accessories_link.stl" scale="${scale}" />
+        <mesh filename="package://waver_description/meshes/accessories_link.stl" scale="${scale}" />
       </geometry>
     </collision>
@@ -74,10 +77,11 @@
       <mass value="${mass_acces1}" />
       <origin xyz="${mass_center_acces1}" rpy="0 0 ${pi/2}" />
-      <inertia ixx="1.8160055789601745e-07" iyy="8.100907081280738e-07" izz="8.100806017664777e-07" ixy="0.0" iyz="0.0" ixz="0.0" />
+      <inertia ixx="8.4505377139432e-14" iyy="3.769648155305237e-13" izz="3.769601126710828e-13"
+        ixy="0.0" iyz="0.0" ixz="0.0" />
     </inertial>
     <visual>
       <origin xyz="${position_acces1}" rpy="0 0 ${pi/2}" />
       <geometry>
-        <mesh filename="file:///$(find waver_description)/meshes/accessories1_link.stl" scale="${scale}" />
+        <mesh filename="package://waver_description/meshes/accessories1_link.stl" scale="${scale}" />
       </geometry>
       <xacro:black_material />
@@ -86,5 +90,5 @@
       <origin xyz="${position_acces1}" rpy="0 0 ${pi/2}" />
       <geometry>
-        <mesh filename="file:///$(find waver_description)/meshes/accessories1_link.stl" scale="${scale}" />
+        <mesh filename="package://waver_description/meshes/accessories1_link.stl" scale="${scale}" />
       </geometry>
     </collision>
@@ -94,10 +98,11 @@
       <mass value="${mass_screen}" />
       <origin xyz="${mass_center_screen}" rpy="0 0 ${pi/2}" />
-      <inertia ixx="3.186534864702538e-08" iyy="2.5666330224105178e-07" izz="2.7215400443770056e-07" ixy="0.0" iyz="0.0" ixz="0.0" />
+      <inertia ixx="2.2613546657562738e-14" iyy="1.821435448519393e-13" izz="1.9313666847229008e-13"
+        ixy="0.0" iyz="0.0" ixz="0.0" />
     </inertial>
     <visual>
       <origin xyz="${position_screen}" rpy="0 0 ${pi/2}" />
       <geometry>
-        <mesh filename="file:///$(find waver_description)/meshes/oled_screen_link.stl" scale="${scale}" />
+        <mesh filename="package://waver_description/meshes/oled_screen_link.stl" scale="${scale}" />
       </geometry>
       <xacro:dark_blue_material />
@@ -106,5 +111,5 @@
       <origin xyz="${position_screen}" rpy="0 0 ${pi/2}" />
       <geometry>
-        <mesh filename="file:///$(find waver_description)/meshes/oled_screen_link.stl" scale="${scale}" />
+        <mesh filename="package://waver_description/meshes/oled_screen_link.stl" scale="${scale}" />
       </geometry>
     </collision>
@@ -114,10 +119,12 @@
       <mass value="${mass_wbl}" />
       <origin xyz="0 0 0" rpy="0 0 ${pi/2}" />
-      <inertia ixx="0.0011153598236428852" iyy="0.0007115715475157099" izz="0.0007099489539679392" ixy="0.0" iyz="0.0" ixz="0.0" />
+      <inertia ixx="6.689307761499951e-05" iyy="4.2676101388344066e-05" izz="4.2578787253633605e-05"
+        ixy="0.0" iyz="0.0" ixz="0.0" />
     </inertial>
     <visual>
       <origin xyz="${position_wbl}" rpy="0 0 ${pi/2}" />
       <geometry>
-        <mesh filename="file:///$(find waver_description)/meshes/wheel_back_left_link.stl" scale="${scale}" />
+        <mesh filename="package://waver_description/meshes/wheel_back_left_link.stl"
+          scale="${scale}" />
       </geometry>
       <xacro:black_material />
@@ -126,5 +133,6 @@
       <origin xyz="${position_wbl}" rpy="0 0 ${pi/2}" />
       <geometry>
-        <mesh filename="file:///$(find waver_description)/meshes/wheel_back_left_link.stl" scale="${scale}" />
+        <mesh filename="package://waver_description/meshes/wheel_back_left_link.stl"
+          scale="${scale}" />
       </geometry>
     </collision>
@@ -134,10 +142,12 @@
       <mass value="${mass_wfl}" />
       <origin xyz="0 0 0" rpy="0 0 ${pi/2}" />
-      <inertia ixx="0.0011153598236428852" iyy="0.0007115715475157099" izz="0.0007099489539679392" ixy="0.0" iyz="0.0" ixz="0.0" />
+      <inertia ixx="6.6894731155928e-05" iyy="4.2676101388344066e-05" izz="4.2580440794562095e-05"
+        ixy="0.0" iyz="0.0" ixz="0.0" />
     </inertial>
     <visual>
       <origin xyz="${position_wfl}" rpy="0 0 ${pi/2}" />
       <geometry>
-        <mesh filename="file:///$(find waver_description)/meshes/wheel_front_left_link.stl" scale="${scale}" />
+        <mesh filename="package://waver_description/meshes/wheel_front_left_link.stl"
+          scale="${scale}" />
       </geometry>
       <xacro:black_material />
@@ -146,5 +156,6 @@
       <origin xyz="${position_wfl}" rpy="0 0 ${pi/2}" />
       <geometry>
-        <mesh filename="file:///$(find waver_description)/meshes/wheel_front_left_link.stl" scale="${scale}" />
+        <mesh filename="package://waver_description/meshes/wheel_front_left_link.stl"
+          scale="${scale}" />
       </geometry>
     </collision>
@@ -154,10 +165,12 @@
       <mass value="${mass_wfr}" />
       <origin xyz="0 0 0" rpy="0 0 ${pi/2}" />
-      <inertia ixx="0.0011153598236428852" iyy="0.0007115715475157099" izz="0.0007099489539679392" ixy="0.0" iyz="0.0" ixz="0.0" />
+      <inertia ixx="6.689307761499951e-05" iyy="4.267610303653357e-05" izz="4.2578788901823125e-05"
+        ixy="0.0" iyz="0.0" ixz="0.0" />
     </inertial>
     <visual>
       <origin xyz="${position_wfr}" rpy="0 0 ${pi/2}" />
       <geometry>
-        <mesh filename="file:///$(find waver_description)/meshes/wheel_front_right_link.stl" scale="${scale}" />
+        <mesh filename="package://waver_description/meshes/wheel_front_right_link.stl"
+          scale="${scale}" />
       </geometry>
       <xacro:black_material />
@@ -166,5 +179,6 @@
       <origin xyz="${position_wfr}" rpy="0 0 ${pi/2}" />
       <geometry>
-        <mesh filename="file:///$(find waver_description)/meshes/wheel_front_right_link.stl" scale="${scale}" />
+        <mesh filename="package://waver_description/meshes/wheel_front_right_link.stl"
+          scale="${scale}" />
       </geometry>
     </collision>
@@ -174,10 +188,12 @@
       <mass value="${mass_wbr}" />
       <origin xyz="0 0 0" rpy="0 0 ${pi/2}" />
-      <inertia ixx="0.0011153598236428852" iyy="0.0007115715475157099" izz="0.0007099489539679392" ixy="0.0" iyz="0.0" ixz="0.0" />
+      <inertia ixx="6.6894731155928e-05" iyy="4.267610303653357e-05" izz="4.25804424427516e-05"
+        ixy="0.0" iyz="0.0" ixz="0.0" />
     </inertial>
     <visual>
       <origin xyz="${position_wbr}" rpy="0 0 ${pi/2}" />
       <geometry>
-        <mesh filename="file:///$(find waver_description)/meshes/wheel_back_right_link.stl" scale="${scale}" />
+        <mesh filename="package://waver_description/meshes/wheel_back_right_link.stl"
+          scale="${scale}" />
       </geometry>
       <xacro:black_material />
@@ -186,5 +202,6 @@
       <origin xyz="${position_wbr}" rpy="0 0 ${pi/2}" />
       <geometry>
-        <mesh filename="file:///$(find waver_description)/meshes/wheel_back_right_link.stl" scale="${scale}" />
+        <mesh filename="package://waver_description/meshes/wheel_back_right_link.stl"
+          scale="${scale}" />
       </geometry>
     </collision>
@@ -207,5 +224,5 @@
     <child link="accessories_link" />
   </joint>
-<joint name="top_acces1_joint" type="fixed">
+  <joint name="top_acces1_joint" type="fixed">
     <origin xyz="${positions_acces1_joint}" rpy="0 0 0" />
     <parent link="top_shell_link" />
