Commit message: chore: inverting rotations for right wheels

File: urdf/waver.xacro (robot description, xacro)
@@ -229,14 +229,14 @@
   </joint>
   <joint name="wheel_front_right_joint" type="continuous">
-    <origin xyz="${position_wfr_joint}" rpy="0 0 0" />
+    <origin xyz="${position_wfr_joint}" rpy="0 0 ${pi}" />
     <parent link="base_link" />
     <child link="wheel_front_right_link" />
-    <axis xyz="0 1 0" />
+    <axis xyz="0 -1 0" />
   </joint>
   <joint name="wheel_back_right_joint" type="continuous">
-    <origin xyz="${position_wbr_joint}" rpy="0 0 0" />
+    <origin xyz="${position_wbr_joint}" rpy="0 0 ${pi}" />
     <parent link="base_link" />
     <child link="wheel_back_right_link" />
-    <axis xyz="0 1 0" />
+    <axis xyz="0 -1 0" />
   </joint>
 </robot>

Commit message: fix: filename updated

File: urdf/waver.xacro (robot description, xacro)
@@ -20,5 +20,5 @@
       <origin xyz="0 0 0" rpy="0 0 ${pi/2}" />
       <geometry>
-        <mesh filename="package://waver_description/meshes/base_link.stl" scale="${scale}" />
+        <mesh filename="file:///$(find waver_description)/meshes/base_link.stl" scale="${scale}" />
       </geometry>
       <xacro:dark_gray_material />
@@ -27,5 +27,5 @@
       <origin xyz="0 0 0" rpy="0 0 ${pi/2}" />
       <geometry>
-        <mesh filename="package://waver_description/meshes/base_link.stl" scale="${scale}" />
+        <mesh filename="file:///$(find waver_description)/meshes/base_link.stl" scale="${scale}" />
       </geometry>
     </collision>
@@ -41,5 +41,5 @@
       <origin xyz="0 0 0" rpy="0 0 ${pi/2}" />
       <geometry>
-        <mesh filename="package://waver_description/meshes/top_shell_link.stl" scale="${scale}" />
+        <mesh filename="file:///$(find waver_description)/meshes/top_shell_link.stl" scale="${scale}" />
       </geometry>
       <xacro:dark_gray_material />
@@ -48,5 +48,5 @@
       <origin xyz="0 0 0" rpy="0 0 ${pi/2}" />
       <geometry>
-        <mesh filename="package://waver_description/meshes/top_shell_link.stl" scale="${scale}" />
+        <mesh filename="file:///$(find waver_description)/meshes/top_shell_link.stl" scale="${scale}" />
       </geometry>
     </collision>
@@ -62,5 +62,5 @@
       <origin xyz="${position_acces}" rpy="0 0 ${pi/2}" />
       <geometry>
-        <mesh filename="package://waver_description/meshes/accessories_link.stl" scale="${scale}" />
+        <mesh filename="file:///$(find waver_description)/meshes/accessories_link.stl" scale="${scale}" />
       </geometry>
       <xacro:black_material />
@@ -69,5 +69,5 @@
       <origin xyz="${position_acces}" rpy="0 0 ${pi/2}" />
       <geometry>
-        <mesh filename="package://waver_description/meshes/accessories_link.stl" scale="${scale}" />
+        <mesh filename="file:///$(find waver_description)/meshes/accessories_link.stl" scale="${scale}" />
       </geometry>
     </collision>
@@ -83,5 +83,5 @@
       <origin xyz="${position_acces1}" rpy="0 0 ${pi/2}" />
       <geometry>
-        <mesh filename="package://waver_description/meshes/accessories1_link.stl" scale="${scale}" />
+        <mesh filename="file:///$(find waver_description)/meshes/accessories1_link.stl" scale="${scale}" />
       </geometry>
       <xacro:black_material />
@@ -90,5 +90,5 @@
       <origin xyz="${position_acces1}" rpy="0 0 ${pi/2}" />
       <geometry>
-        <mesh filename="package://waver_description/meshes/accessories1_link.stl" scale="${scale}" />
+        <mesh filename="file:///$(find waver_description)/meshes/accessories1_link.stl" scale="${scale}" />
       </geometry>
     </collision>
@@ -104,5 +104,5 @@
       <origin xyz="${position_screen}" rpy="0 0 ${pi/2}" />
       <geometry>
-        <mesh filename="package://waver_description/meshes/oled_screen_link.stl" scale="${scale}" />
+        <mesh filename="file:///$(find waver_description)/meshes/oled_screen_link.stl" scale="${scale}" />
       </geometry>
       <xacro:dark_blue_material />
@@ -111,5 +111,5 @@
       <origin xyz="${position_screen}" rpy="0 0 ${pi/2}" />
       <geometry>
-        <mesh filename="package://waver_description/meshes/oled_screen_link.stl" scale="${scale}" />
+        <mesh filename="file:///$(find waver_description)/meshes/oled_screen_link.stl" scale="${scale}" />
       </geometry>
     </collision>
@@ -125,5 +125,5 @@
       <origin xyz="${position_wbl}" rpy="0 0 ${pi/2}" />
       <geometry>
-        <mesh filename="package://waver_description/meshes/wheel_back_left_link.stl"
+        <mesh filename="file:///$(find waver_description)/meshes/wheel_back_left_link.stl"
           scale="${scale}" />
       </geometry>
@@ -133,5 +133,5 @@
       <origin xyz="${position_wbl}" rpy="0 0 ${pi/2}" />
       <geometry>
-        <mesh filename="package://waver_description/meshes/wheel_back_left_link.stl"
+        <mesh filename="file:///$(find waver_description)/meshes/wheel_back_left_link.stl"
           scale="${scale}" />
       </geometry>
@@ -148,5 +148,5 @@
       <origin xyz="${position_wfl}" rpy="0 0 ${pi/2}" />
       <geometry>
-        <mesh filename="package://waver_description/meshes/wheel_front_left_link.stl"
+        <mesh filename="file:///$(find waver_description)/meshes/wheel_front_left_link.stl"
           scale="${scale}" />
       </geometry>
@@ -156,5 +156,5 @@
       <origin xyz="${position_wfl}" rpy="0 0 ${pi/2}" />
       <geometry>
-        <mesh filename="package://waver_description/meshes/wheel_front_left_link.stl"
+        <mesh filename="file:///$(find waver_description)/meshes/wheel_front_left_link.stl"
           scale="${scale}" />
       </geometry>
@@ -171,5 +171,5 @@
       <origin xyz="${position_wfr}" rpy="0 0 ${pi/2}" />
       <geometry>
-        <mesh filename="package://waver_description/meshes/wheel_front_right_link.stl"
+        <mesh filename="file:///$(find waver_description)/meshes/wheel_front_right_link.stl"
           scale="${scale}" />
       </geometry>
@@ -179,5 +179,5 @@
       <origin xyz="${position_wfr}" rpy="0 0 ${pi/2}" />
       <geometry>
-        <mesh filename="package://waver_description/meshes/wheel_front_right_link.stl"
+        <mesh filename="file:///$(find waver_description)/meshes/wheel_front_right_link.stl"
           scale="${scale}" />
       </geometry>
@@ -194,5 +194,5 @@
       <origin xyz="${position_wbr}" rpy="0 0 ${pi/2}" />
       <geometry>
-        <mesh filename="package://waver_description/meshes/wheel_back_right_link.stl"
+        <mesh filename="file:///$(find waver_description)/meshes/wheel_back_right_link.stl"
           scale="${scale}" />
       </geometry>
@@ -202,5 +202,5 @@
       <origin xyz="${position_wbr}" rpy="0 0 ${pi/2}" />
       <geometry>
-        <mesh filename="package://waver_description/meshes/wheel_back_right_link.stl"
+        <mesh filename="file:///$(find waver_description)/meshes/wheel_back_right_link.stl"
           scale="${scale}" />
       </geometry>
